File: ControlChips.kicad_sch (KiCad schematic)
At the start: 22 parts, among them J13 STM_Prog, J16 Conn_01x04_Socket, J18 Conn_01x03_Pin, J2 Conn_01x15_Socket, J26 Conn_01x06_Socket, J27 USB_B_Micro, J3 Conn_01x15_Socket, J5 Conn_01x08_Socket, U14 ATmega328P-A, U5 ATmega328P-P, U6 STM32F103R8Tx

Commit message: Release 1.0
Parts:
- added C8, C9: 22p, Capacitor_THT:C_Rect_L7.0mm_W3.5mm_P5.00mm, symbol Device:C
Connections:
- net GND: now also C8.2, C9.1
- net OSC_A: now also C9.2
- net OSC_B: now also C8.1
Other:
- note added: "CONTROL block"
- note added: "You can use any of these chips, but only one chip and only one voltage regulator. The STM32 blocks PA, PB and a few of the PC pins provided need to be manually soldered to the output pins of the ESP32 socket. They digital outputs for the 6 MOSFETs are hard wired in the PCB only for ESP32 and the Atmega chips. For STM32 we have more flexibility. USB-B micro port is used to program STM32 only. ESP3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"
- moved on the sheet: C5, C6, C7, J13, J16, J18, J2, J26, J27, J3, J5, OSC1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

Commit message: Release 1.1
Parts:
- added C10, C11: 100n, Capacitor_THT:C_Rect_L7.0mm_W3.5mm_P5.00mm, symbol Device:C
- added J28: USB_C_adapter, Connector_PinSocket_2.54mm:PinSocket_1x04_P2.54mm_Vertical, symbol Connector:Conn_01x04_Socket
- added J29: USB_C_Receptacle_USB2.0_16P, Connector_USB:USB_C_Receptacle_GCT_USB4085, symbol Connector:USB_C_Receptacle_USB2.0_16P
- added OSC3: Crystal, Crystal:Crystal_HC49-U_Vertical, symbol Device:Crystal
- added R23, R24: 5.1k, Diode_SMD:D_2512_6332Metric, symbol Device:R
- added R23Alt2, R24alt2: 2.1k, TO220:R_Axial_Clean, symbol Device:R
- added R23alt1, R24alt1: 3k, TO220:R_Axial_Clean, symbol Device:R
- added TTL_Socket1, TTL_Socket2: Conn_01x06_Socket, Connector_PinSocket_2.54mm:PinSocket_1x06_P2.54mm_Vertical, symbol Connector:Conn_01x06_Socket
Connections:
- net 3V3: now also TTL_Socket1.6 (Pin_6)
- net GND: now also C10.2, C11.2, J28.4 (Pin_4), J29.A1 (GND), J29.A12 (GND), J29.B1 (GND), J29.B12 (GND), J29.S1 (SHIELD), R23.1, R23Alt2.1, R24.1, R24alt2.1, TTL_Socket1.1 (Pin_1)
- net OSC_C: no longer U6.5 (PD0)
- net OSC_D: no longer U6.6 (PD1)
- net PA11_D+: now also J28.3 (Pin_3), J29.A6 (D+), J29.B6 (D+)
- net PA11_D-: now also J28.2 (Pin_2), J29.A7 (D-), J29.B7 (D-)
- net Rx: now also TTL_Socket1.4 (Pin_4)
- net Tx: now also TTL_Socket1.3 (Pin_3)
- net VDC: now also J28.1 (Pin_1), J29.A4 (VBUS), J29.A9 (VBUS), J29.B4 (VBUS), J29.B9 (VBUS)
- new net: J29.A5 (CC1), R23.2, R23alt1.2
- new net: J29.B5 (CC2), R24.2, R24alt1.2
- new net: R24alt1.1, R24alt2.2
- new net: R23Alt2.2, R23alt1.1
- new net 5V: TTL_Socket1.2 (Pin_2)
- new net DTR: TTL_Socket1.5 (Pin_5)
- new net OSC_C2: C11.1, OSC3.2, U6.5 (PD0)
- new net OSC_D2: C10.1, OSC3.1, U6.6 (PD1)
- no-connect marks 17 -> 19
Other:
- moved on the sheet: R22

Commit message: Release 1.2
Parts:
- C10, C11, C5, C6, C7, C8, C9: footprint Capacitor_THT:C_Rect_L7.0mm_W3.5mm_P5.00mm -> Project_Footprints:C_Rect_L7.0mm_W3.5mm_P5.00mm
- J13, J16, J28: footprint Connector_PinSocket_2.54mm:PinSocket_1x04_P2.54mm_Vertical -> Project_Footprints:PinSocket_1x04_P2.54mm_Vertical
- J18, ProgramMode1: footprint Connector_PinHeader_2.54mm:PinHeader_1x03_P2.54mm_Vertical -> Project_Footprints:PinHeader_1x03_P2.54mm_Vertical
- J2, J3: footprint Connector_PinSocket_2.54mm:PinSocket_1x15_P2.54mm_Vertical -> Project_Footprints:PinSocket_1x15_P2.54mm_Vertical
- J26, TTL_Socket1, TTL_Socket2: footprint Connector_PinSocket_2.54mm:PinSocket_1x06_P2.54mm_Vertical -> Project_Footprints:PinSocket_1x06_P2.54mm_Vertical
- J27: footprint Connector_USB:USB_Micro-B_Wuerth_629105150521 -> Project_Footprints:USB_Micro-B_Wuerth_629105150521
- J29: footprint Connector_USB:USB_C_Receptacle_GCT_USB4085 -> Project_Footprints:USB_C_Receptacle_GCT_USB4085
- J5: footprint Connector_PinSocket_2.54mm:PinSocket_1x08_P2.54mm_Vertical -> Project_Footprints:PinSocket_1x08_P2.54mm_Vertical
- OSC1, OSC2, OSC3: footprint Crystal:Crystal_HC49-U_Vertical -> Project_Footprints:Crystal_HC49-U_Vertical
- PA_Socket1, PB_Socket1: footprint Connector_PinSocket_2.54mm:PinSocket_1x16_P2.54mm_Vertical -> Project_Footprints:PinSocket_1x16_P2.54mm_Vertical
- R20, R21, R22, R23Alt2, R23alt1, R24alt1, R24alt2: footprint TO220:R_Axial_Clean -> Project_Footprints:R_Axial_Clean
- R23, R24: footprint Diode_SMD:D_2512_6332Metric -> Project_Footprints:D_2512_6332Metric
- U14: footprint termocuplu:TQFP-32_SLIM -> Project_Footprints:TQFP-32_SLIM
- U5: footprint Package_DIP:DIP-28_W7.62mm_Socket -> Project_Footprints:DIP-28_W7.62mm_Socket
- U6: footprint Package_QFP:LQFP-64_10x10mm_P0.5mm -> Project_Footprints:LQFP-64_10x10mm_P0.5mm
Changed lines of the file:
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@@
 			)
 		)
-		(property "Footprint" "Connector_PinSocket_2.54mm:PinSocket_1x06_P2.54mm_Vertical"
+		(property "Footprint" "Project_Footprints:PinSocket_1x06_P2.54mm_Vertical"
 			(at 69.85 166.37 0)
 			(effects
@@
 			)
 		)
-		(property "Footprint" "Crystal:Crystal_HC49-U_Vertical"
+		(property "Footprint" "Project_Footprints:Crystal_HC49-U_Vertical"
 			(at 271.78 160.02 0)
 			(effects
@@
 			)
 		)
-		(property "Footprint" "Capacitor_THT:C_Rect_L7.0mm_W3.5mm_P5.00mm"
+		(property "Footprint" "Project_Footprints:C_Rect_L7.0mm_W3.5mm_P5.00mm"
 			(at 321.0052 177.8 0)
 			(effects
@@
 			)
 		)
-		(property "Footprint" "Connector_USB:USB_C_Receptacle_GCT_USB4085"
+		(property "Footprint" "Project_Footprints:USB_C_Receptacle_GCT_USB4085"
 			(at 153.67 228.6 0)
 			(effects
@@
 			)
 		)
-		(property "Footprint" "Capacitor_THT:C_Rect_L7.0mm_W3.5mm_P5.00mm"
+		(property "Footprint" "Project_Footprints:C_Rect_L7.0mm_W3.5mm_P5.00mm"
 			(at 290.5252 161.29 0)
 			(effects
@@
 			)
 		)
-		(property "Footprint" "TO220:R_Axial_Clean"
+		(property "Footprint" "Project_Footprints:R_Axial_Clean"
 			(at 190.5 231.902 90)
 			(effects
@@
 			)
 		)
-		(property "Footprint" "Connector_PinHeader_2.54mm:PinHeader_1x03_P2.54mm_Vertical"
+		(property "Footprint" "Project_Footprints:PinHeader_1x03_P2.54mm_Vertical"
 			(at 256.54 69.85 0)
 			(effects
@@
 			)
 		)
-		(property "Footprint" "Connector_PinSocket_2.54mm:PinSocket_1x06_P2.54mm_Vertical"
+		(property "Footprint" "Project_Footprints:PinSocket_1x06_P2.54mm_Vertical"
 			(at 50.8 182.88 0)
 			(effects
@@
 			)
 		)
-		(property "Footprint" "Connector_USB:USB_Micro-B_Wuerth_629105150521"
+		(property "Footprint" "Project_Footprints:USB_Micro-B_Wuerth_629105150521"
 			(at 146.05 151.13 0)
 			(effects
@@
 			)
 		)
-		(property "Footprint" "Connector_PinSocket_2.54mm:PinSocket_1x06_P2.54mm_Vertical"
+		(property "Footprint" "Project_Footprints:PinSocket_1x06_P2.54mm_Vertical"
 			(at 35.56 190.5 0)
 			(effects
@@
 			)
 		)
-		(property "Footprint" "Package_DIP:DIP-28_W7.62mm_Socket"
+		(property "Footprint" "Project_Footprints:DIP-28_W7.62mm_Socket"
 			(at 173.99 92.71 0)
 			(effects
@@
 			)
 		)
-		(property "Footprint" "Diode_SMD:D_2512_6332Metric"
+		(property "Footprint" "Project_Footprints:D_2512_6332Metric"
 			(at 175.26 216.662 90)
 			(effects
@@
 			)
 		)
-		(property "Footprint" "TO220:R_Axial_Clean"
+		(property "Footprint" "Project_Footprints:R_Axial_Clean"
 			(at 187.96 212.852 90)
 			(effects
@@
 			)
 		)
-		(property "Footprint" "Crystal:Crystal_HC49-U_Vertical"
+		(property "Footprint" "Project_Footprints:Crystal_HC49-U_Vertical"
 			(at 328.93 162.56 0)
 			(effects
@@
 			)
 		)
-		(property "Footprint" "termocuplu:TQFP-32_SLIM"
+		(property "Footprint" "Project_Footprints:TQFP-32_SLIM"
 			(at 293.37 92.71 0)
 			(effects
@@
 			)
 		)
-		(property "Footprint" "Capacitor_THT:C_Rect_L7.0mm_W3.5mm_P5.00mm"
+		(property "Footprint" "Project_Footprints:C_Rect_L7.0mm_W3.5mm_P5.00mm"
 			(at 145.7452 110.49 0)
 			(effects
@@
 			)
 		)
-		(property "Footprint" "Capacitor_THT:C_Rect_L7.0mm_W3.5mm_P5.00mm"
+		(property "Footprint" "Project_Footprints:C_Rect_L7.0mm_W3.5mm_P5.00mm"
 			(at 145.7452 90.17 0)
 			(effects
@@
 			)
 		)
-		(property "Footprint" "Capacitor_THT:C_Rect_L7.0mm_W3.5mm_P5.00mm"
+		(property "Footprint" "Project_Footprints:C_Rect_L7.0mm_W3.5mm_P5.00mm"
 			(at 347.6752 163.83 0)
 			(effects
@@
 			)
 		)
-		(property "Footprint" "Diode_SMD:D_2512_6332Metric"
+		(property "Footprint" "Project_Footprints:D_2512_6332Metric"
 			(at 175.26 219.202 90)
 			(effects
@@
 			)
 		)
-		(property "Footprint" "Connector_PinHeader_2.54mm:PinHeader_1x03_P2.54mm_Vertical"
+		(property "Footprint" "Project_Footprints:PinHeader_1x03_P2.54mm_Vertical"
 			(at 58.42 123.19 0)
 			(effects
@@
 			)
 		)
-		(property "Footprint" "Connector_PinSocket_2.54mm:PinSocket_1x04_P2.54mm_Vertical"
+		(property "Footprint" "Project_Footprints:PinSocket_1x04_P2.54mm_Vertical"
 			(at 259.08 147.32 0)
 			(effects
@@
 			)
 		)
-		(property "Footprint" "TO220:R_Axial_Clean"
+		(property "Footprint" "Project_Footprints:R_Axial_Clean"
 			(at 200.66 231.902 90)
 			(effects
@@
 			)
 		)
-		(property "Footprint" "TO220:R_Axial_Clean"
+		(property "Footprint" "Project_Footprints:R_Axial_Clean"
 			(at 198.12 212.852 90)
 			(effects
@@
 			)
 		)
-		(property "Footprint" "TO220:R_Axial_Clean"
+		(property "Footprint" "Project_Footprints:R_Axial_Clean"
 			(at 80.01 139.192 90)
 			(effects
@@
 			)
 		)
-		(property "Footprint" "TO220:R_Axial_Clean"
+		(property "Footprint" "Project_Footprints:R_Axial_Clean"
 			(at 175.768 161.29 90)
 			(effects
@@
 			)
 		)
-		(property "Footprint" "Crystal:Crystal_HC49-U_Vertical"
+		(property "Footprint" "Project_Footprints:Crystal_HC49-U_Vertical"
 			(at 146.05 95.25 0)
 			(effects
@@
 			)
 		)
-		(property "Footprint" "Package_QFP:LQFP-64_10x10mm_P0.5mm"
+		(property "Footprint" "Project_Footprints:LQFP-64_10x10mm_P0.5mm"
 			(at 87.63 222.25 0)
 			(effects
@@
 			)
 		)
-		(property "Footprint" "Connector_PinSocket_2.54mm:PinSocket_1x15_P2.54mm_Vertical"
+		(property "Footprint" "Project_Footprints:PinSocket_1x15_P2.54mm_Vertical"
 			(at 106.68 78.74 0)
 			(effects
@@
 			)
 		)
-		(property "Footprint" "Connector_PinSocket_2.54mm:PinSocket_1x04_P2.54mm_Vertical"
+		(property "Footprint" "Project_Footprints:PinSocket_1x04_P2.54mm_Vertical"
 			(at 232.41 106.68 0)
 			(effects
@@
 			)
 		)
-		(property "Footprint" "Connector_PinSocket_2.54mm:PinSocket_1x15_P2.54mm_Vertical"
+		(property "Footprint" "Project_Footprints:PinSocket_1x15_P2.54mm_Vertical"
 			(at 87.63 78.74 0)
 			(effects
@@
 			)
 		)
-		(property "Footprint" "Capacitor_THT:C_Rect_L7.0mm_W3.5mm_P5.00mm"
+		(property "Footprint" "Project_Footprints:C_Rect_L7.0mm_W3.5mm_P5.00mm"
 			(at 263.8552 175.26 0)
 			(effects
@@
 			)
 		)
-		(property "Footprint" "Connector_PinSocket_2.54mm:PinSocket_1x04_P2.54mm_Vertical"
+		(property "Footprint" "Project_Footprints:PinSocket_1x04_P2.54mm_Vertical"
 			(at 193.04 144.78 0)
 			(effects
@@
 			)
 		)
-		(property "Footprint" "Connector_PinSocket_2.54mm:PinSocket_1x16_P2.54mm_Vertical"
+		(property "Footprint" "Project_Footprints:PinSocket_1x16_P2.54mm_Vertical"
 			(at 217.17 152.4 0)
 			(effects
@@
 			)
 		)
-		(property "Footprint" "TO220:R_Axial_Clean"
+		(property "Footprint" "Project_Footprints:R_Axial_Clean"
 			(at 201.93 102.108 90)
 			(effects
@@
 			)
 		)
-		(property "Footprint" "Capacitor_THT:C_Rect_L7.0mm_W3.5mm_P5.00mm"
+		(property "Footprint" "Project_Footprints:C_Rect_L7.0mm_W3.5mm_P5.00mm"
 			(at 63.1952 143.51 0)
 			(effects
@@
 			)
 		)
-		(property "Footprint" "Connector_PinSocket_2.54mm:PinSocket_1x08_P2.54mm_Vertical"
+		(property "Footprint" "Project_Footprints:PinSocket_1x08_P2.54mm_Vertical"
 			(at 66.04 76.2 0)
 			(effects
@@
 			)
 		)
-		(property "Footprint" "Connector_PinSocket_2.54mm:PinSocket_1x16_P2.54mm_Vertical"
+		(property "Footprint" "Project_Footprints:PinSocket_1x16_P2.54mm_Vertical"
 			(at 187.96 187.96 0)
 			(effects
