File: ESP_IOBoard_V4.kicad_sch (KiCad schematic)
At the start: 10 parts

Commit message: Release 1.2
Parts:
- H1, H10, H2, H3, H4, H5, H6, H7, H8, H9: footprint MountingHole:MountingHole_2.7mm_M2.5_Pad_Via -> Project_Footprints:MountingHole_2.7mm_M2.5_Pad_Via
Changed lines of the file:
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@@
 			)
 		)
-		(property "Footprint" "MountingHole:MountingHole_2.7mm_M2.5_Pad_Via"
+		(property "Footprint" "Project_Footprints:MountingHole_2.7mm_M2.5_Pad_Via"
 			(at 27.94 113.03 0)
 			(effects
@@
 			)
 		)
-		(property "Footprint" "MountingHole:MountingHole_2.7mm_M2.5_Pad_Via"
+		(property "Footprint" "Project_Footprints:MountingHole_2.7mm_M2.5_Pad_Via"
 			(at 78.74 92.71 0)
 			(effects
@@
 			)
 		)
-		(property "Footprint" "MountingHole:MountingHole_2.7mm_M2.5_Pad_Via"
+		(property "Footprint" "Project_Footprints:MountingHole_2.7mm_M2.5_Pad_Via"
 			(at 128.27 92.71 0)
 			(effects
@@
 			)
 		)
-		(property "Footprint" "MountingHole:MountingHole_2.7mm_M2.5_Pad_Via"
+		(property "Footprint" "Project_Footprints:MountingHole_2.7mm_M2.5_Pad_Via"
 			(at 85.09 129.54 0)
 			(effects
@@
 			)
 		)
-		(property "Footprint" "MountingHole:MountingHole_2.7mm_M2.5_Pad_Via"
+		(property "Footprint" "Project_Footprints:MountingHole_2.7mm_M2.5_Pad_Via"
 			(at 26.67 92.71 0)
 			(effects
@@
 			)
 		)
-		(property "Footprint" "MountingHole:MountingHole_2.7mm_M2.5_Pad_Via"
+		(property "Footprint" "Project_Footprints:MountingHole_2.7mm_M2.5_Pad_Via"
 			(at 86.36 113.03 0)
 			(effects
@@
 			)
 		)
-		(property "Footprint" "MountingHole:MountingHole_2.7mm_M2.5_Pad_Via"
+		(property "Footprint" "Project_Footprints:MountingHole_2.7mm_M2.5_Pad_Via"
 			(at 111.76 129.54 0)
 			(effects
@@
 			)
 		)
-		(property "Footprint" "MountingHole:MountingHole_2.7mm_M2.5_Pad_Via"
+		(property "Footprint" "Project_Footprints:MountingHole_2.7mm_M2.5_Pad_Via"
 			(at 111.76 113.03 0)
 			(effects
@@
 			)
 		)
-		(property "Footprint" "MountingHole:MountingHole_2.7mm_M2.5_Pad_Via"
+		(property "Footprint" "Project_Footprints:MountingHole_2.7mm_M2.5_Pad_Via"
 			(at 105.41 92.71 0)
 			(effects
@@
 			)
 		)
-		(property "Footprint" "MountingHole:MountingHole_2.7mm_M2.5_Pad_Via"
+		(property "Footprint" "Project_Footprints:MountingHole_2.7mm_M2.5_Pad_Via"
 			(at 58.42 113.03 0)
 			(effects
