File: GateDrivers.kicad_sch (KiCad schematic)
At the start: 136 parts, among them J17 Conn_01x07_Socket, J19 Conn_01x07_Socket, J20 Conn_01x07_Socket, J25 Conn_01x08_Socket, Q10 PZT2222A, Q11 PZT2222A, Q12 PZT2222A, Q13 PZT2222A, Q14 PZT2222A, Q15 PZT2222A, Q16 PZT2222A, Q17 PZT2222A, Q18 PZT2222A, Q19 BCP51, Q20 BCP51, Q21 BCP51, Q22 BCP51, Q23 BCP51, Q24 BCP51, Q25 PZT2222A, Q26 PZT2222A, Q27 PZT2222A, Q28 PZT2222A, Q29 PZT2222A, Q30 PZT2222A, Q6 PZT2222A, Q8 PZT2222A, Q9 PZT2222A, U1 PC817, U10 PC817, U12 PC817, U2 PC817, U8 PC817, U9 PC817

Commit message: Release 1.0
Other:
- note added: "For each of the 6 output MOSFETs: - connect digital signals (GateDriveN) directly to GatedriveN_HI outputs and bypass the gate driver entirely, but only if using logic level MOSFETs - otherwise, for MOSFETs that don't open fully at 3.3V or 5V, for each channel the board allows one of the following options. Use what you can: - UCC27511ADBV dedicated IC (primary option) OR - PC817 optocoupler (seco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"
- note added: "GATE DRIVERS block"
Changed lines of the file:
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@@
 		)
 	)
+	(text "For each of the 6 output MOSFETs:\n- connect digital signals (GateDriveN) directly to GatedriveN_HI outputs and\nbypass the gate driver entirely, but only if using logic level MOSFETs\n- otherwise, for MOSFETs that don't open fully at 3.3V or 5V, for each\nchannel the board allows one of the following options. \nUse what you can:\n   - UCC27511ADBV dedicated IC (primary option) OR\n   - PC817 optocoupler (second option) OR\n   - Totem pole circuit with TO-92 transistors\n   - Totem pole circuit with TO-223 transistors\nUse whatever you can find. This board is designed for flexibility"
+		(exclude_from_sim no)
+		(at 167.386 353.314 0)
+		(effects
+			(font
+				(size 2.54 2.54)
+				(thickness 0.508)
+				(bold yes)
+			)
+			(justify left)
+		)
+	)
 	(text "UCC27511 gate driver option (primary)\n"
 		(exclude_from_sim no)
@@
 		)
 	)
+	(text "GATE DRIVERS block"
+		(exclude_from_sim no)
+		(at 354.838 228.854 0)
+		(effects
+			(font
+				(size 5.08 5.08)
+				(thickness 1.016)
+				(bold yes)
+			)
+		)
+	)
 	(text "TO92 totem pole option"
 		(exclude_from_sim no)
@@
 		(dnp no)
 		(property "Reference" "Rnpn6"
-			(at 395.224 274.574 90)
+			(at 398.272 280.416 90)
 			(effects
 				(font

Commit message: Release 1.1
Parts:
- removed J25: Conn_01x08_Socket, Connector_PinSocket_2.54mm:PinSocket_1x08_P2.54mm_Vertical, symbol Connector:Conn_01x08_Socket
- removed U1, U10, U12, U2, U8, U9: PC817, TO220:OPTO_NEW, symbol Isolator:PC817
Other:
- note removed: "Optocoupler option (PC817 DIP4)"

Commit message: Release 1.2
Parts:
- 2N3904_1, 2N3904_10, 2N3904_11, 2N3904_12, 2N3904_19, 2N3904_2, 2N3904_20, 2N3904_21, 2N3904_22, 2N3904_23, 2N3904_24, 2N3904_3, 2N3904_4, 2N3904_5, 2N3904_6, 2N3904_7, 2N3904_8, 2N3904_9, BC327_1, BC327_2, BC327_3, BC327_4, BC327_5, BC327_6: footprint TO220:TO-92_Expanded -> Project_Footprints:TO-92_Expanded
- J17, J19, J20: footprint Connector_PinSocket_2.54mm:PinSocket_1x07_P2.54mm_Vertical -> Project_Footprints:PinSocket_1x07_P2.54mm_Vertical
- Q10, Q11, Q12, Q13, Q14, Q15, Q16, Q17, Q18, Q19, Q20, Q21, Q22, Q23, Q24, Q25, Q26, Q27, Q28, Q29, Q30, Q6, Q8, Q9: footprint Package_TO_SOT_SMD:SOT-223-3_TabPin2 -> Project_Footprints:SOT-223-3_TabPin2
- RH5_alt1, RH5_alt10, RH5_alt11, RH5_alt12, RH5_alt13, RH5_alt14, RH5_alt15, RH5_alt16, RH5_alt17, RH5_alt18, RH5_alt19, RH5_alt2, RH5_alt20, RH5_alt21, RH5_alt22, RH5_alt23, RH5_alt24, RH5_alt25, RH5_alt26, RH5_alt27, RH5_alt28, RH5_alt29, RH5_alt3, RH5_alt30, RH5_alt31, RH5_alt32, RH5_alt33, RH5_alt34, RH5_alt35, RH5_alt4, RH5_alt5, RH5_alt6, RH5_alt7, RH5_alt8, RH5_alt9, RL5_alt1: footprint Diode_SMD:D_2512_6332Metric -> Project_Footprints:D_2512_6332Metric
- Rnpn1, Rnpn10, Rnpn11, Rnpn12, Rnpn13, Rnpn14, Rnpn15, Rnpn16, Rnpn17, Rnpn18, Rnpn19, Rnpn2, Rnpn20, Rnpn21, Rnpn22, Rnpn23, Rnpn3, Rnpn33, Rnpn4, Rnpn5, Rnpn6, Rnpn7, Rnpn8, Rnpn9, RoutH_1, RoutH_2, RoutH_3, RoutH_4, RoutH_5, RoutH_6, RoutL_1, RoutL_2, RoutL_3, RoutL_4, RoutL_5, RoutL_6: footprint TO220:R_Axial_Clean -> Project_Footprints:R_Axial_Clean
- UCC27511ADBV_1, UCC27511ADBV_2, UCC27511ADBV_3, UCC27511ADBV_4, UCC27511ADBV_5, UCC27511ADBV_6: footprint Package_TO_SOT_SMD:SOT-23-6 -> Project_Footprints:SOT-23-6
