File: Inputs.kicad_sch (KiCad schematic)
At the start: 26 parts, among them J21 Conn_01x02_Socket, J22 Conn_01x02_Socket, J23 Conn_01x02_Socket, J24 Conn_01x02_Socket, J4 Conn_01x04_Socket, J7 Conn_01x05_Socket, SW1 SW_Push, SW2 SW_Push, SW3 SW_Push, SW4 SW_Push, U4 AD8497

Commit message: Release 1.2
Parts:
- D16_Config1, D17_Config1, TestMode1: footprint Connector_PinHeader_2.54mm:PinHeader_1x03_P2.54mm_Vertical -> Project_Footprints:PinHeader_1x03_P2.54mm_Vertical
- J21, J22, J23, J24: footprint Connector_PinSocket_2.54mm:PinSocket_1x02_P2.54mm_Vertical -> Project_Footprints:PinSocket_1x02_P2.54mm_Vertical
- J4: footprint Connector_PinSocket_2.54mm:PinSocket_1x04_P2.54mm_Vertical -> Project_Footprints:PinSocket_1x04_P2.54mm_Vertical
- J7: footprint Connector_PinSocket_2.54mm:PinSocket_1x05_P2.54mm_Vertical -> Project_Footprints:PinSocket_1x05_P2.54mm_Vertical
- J_T1, J_T2: footprint TerminalBlock:TerminalBlock_bornier-3_P5.08mm -> Project_Footprints:TerminalBlock_bornier-3_P5.08mm
- R19, R28, R29, R33, R35, R37, R38: footprint TO220:R_Axial_Clean -> Project_Footprints:R_Axial_Clean
- R25, R30: footprint Potentiometer_THT:Potentiometer_Piher_PT-6-V_Vertical_Hole -> Project_Footprints:Potentiometer_Piher_PT-6-V_Vertical_Hole
- SW1, SW2, SW3, SW4: footprint Button_Switch_THT:SW_PUSH_6mm -> Project_Footprints:SW_PUSH_6mm
- U3: footprint termocuplu:k type -> Project_Footprints:k type
- U4: footprint Package_SO:MSOP-8_3x3mm_P0.65mm -> Project_Footprints:MSOP-8_3x3mm_P0.65mm
Changed lines of the file:
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@@
 			)
 		)
-		(property "Footprint" "TerminalBlock:TerminalBlock_bornier-3_P5.08mm"
+		(property "Footprint" "Project_Footprints:TerminalBlock_bornier-3_P5.08mm"
 			(at 218.44 81.28 0)
 			(effects
@@
 			)
 		)
-		(property "Footprint" "Potentiometer_THT:Potentiometer_Piher_PT-6-V_Vertical_Hole"
+		(property "Footprint" "Project_Footprints:Potentiometer_Piher_PT-6-V_Vertical_Hole"
 			(at 81.28 47.498 90)
 			(effects
@@
 			)
 		)
-		(property "Footprint" "TO220:R_Axial_Clean"
+		(property "Footprint" "Project_Footprints:R_Axial_Clean"
 			(at 53.34 84.328 90)
 			(effects
@@
 			)
 		)
-		(property "Footprint" "Button_Switch_THT:SW_PUSH_6mm"
+		(property "Footprint" "Project_Footprints:SW_PUSH_6mm"
 			(at 153.67 128.27 0)
 			(effects
@@
 			)
 		)
-		(property "Footprint" "TO220:R_Axial_Clean"
+		(property "Footprint" "Project_Footprints:R_Axial_Clean"
 			(at 215.138 92.71 90)
 			(effects
@@
 			)
 		)
-		(property "Footprint" "TO220:R_Axial_Clean"
+		(property "Footprint" "Project_Footprints:R_Axial_Clean"
 			(at 74.422 52.07 90)
 			(effects
@@
 			)
 		)
-		(property "Footprint" "Potentiometer_THT:Potentiometer_Piher_PT-6-V_Vertical_Hole"
+		(property "Footprint" "Project_Footprints:Potentiometer_Piher_PT-6-V_Vertical_Hole"
 			(at 49.53 46.228 90)
 			(effects
@@
 			)
 		)
-		(property "Footprint" "Connector_PinSocket_2.54mm:PinSocket_1x02_P2.54mm_Vertical"
+		(property "Footprint" "Project_Footprints:PinSocket_1x02_P2.54mm_Vertical"
 			(at 180.34 110.49 0)
 			(effects
@@
 			)
 		)
-		(property "Footprint" "Button_Switch_THT:SW_PUSH_6mm"
+		(property "Footprint" "Project_Footprints:SW_PUSH_6mm"
 			(at 181.61 123.19 0)
 			(effects
@@
 			)
 		)
-		(property "Footprint" "Connector_PinSocket_2.54mm:PinSocket_1x02_P2.54mm_Vertical"
+		(property "Footprint" "Project_Footprints:PinSocket_1x02_P2.54mm_Vertical"
 			(at 212.09 110.49 0)
 			(effects
@@
 			)
 		)
-		(property "Footprint" "termocuplu:k type"
+		(property "Footprint" "Project_Footprints:k type"
 			(at 58.42 119.38 0)
 			(effects
@@
 			)
 		)
-		(property "Footprint" "Connector_PinSocket_2.54mm:PinSocket_1x02_P2.54mm_Vertical"
+		(property "Footprint" "Project_Footprints:PinSocket_1x02_P2.54mm_Vertical"
 			(at 152.4 116.84 0)
 			(effects
@@
 			)
 		)
-		(property "Footprint" "TO220:R_Axial_Clean"
+		(property "Footprint" "Project_Footprints:R_Axial_Clean"
 			(at 60.96 86.868 90)
 			(effects
@@
 			)
 		)
-		(property "Footprint" "TerminalBlock:TerminalBlock_bornier-3_P5.08mm"
+		(property "Footprint" "Project_Footprints:TerminalBlock_bornier-3_P5.08mm"
 			(at 218.44 68.58 0)
 			(effects
@@
 			)
 		)
-		(property "Footprint" "Connector_PinSocket_2.54mm:PinSocket_1x04_P2.54mm_Vertical"
+		(property "Footprint" "Project_Footprints:PinSocket_1x04_P2.54mm_Vertical"
 			(at 34.29 87.63 0)
 			(effects
@@
 			)
 		)
-		(property "Footprint" "Connector_PinSocket_2.54mm:PinSocket_1x02_P2.54mm_Vertical"
+		(property "Footprint" "Project_Footprints:PinSocket_1x02_P2.54mm_Vertical"
 			(at 199.39 140.97 0)
 			(effects
@@
 			)
 		)
-		(property "Footprint" "TO220:R_Axial_Clean"
+		(property "Footprint" "Project_Footprints:R_Axial_Clean"
 			(at 42.672 52.07 90)
 			(effects
@@
 			)
 		)
-		(property "Footprint" "Connector_PinSocket_2.54mm:PinSocket_1x05_P2.54mm_Vertical"
+		(property "Footprint" "Project_Footprints:PinSocket_1x05_P2.54mm_Vertical"
 			(at 124.46 114.3 0)
 			(effects
@@
 			)
 		)
-		(property "Footprint" "TO220:R_Axial_Clean"
+		(property "Footprint" "Project_Footprints:R_Axial_Clean"
 			(at 154.178 74.93 90)
 			(effects
@@
 			)
 		)
-		(property "Footprint" "TO220:R_Axial_Clean"
+		(property "Footprint" "Project_Footprints:R_Axial_Clean"
 			(at 213.868 58.42 90)
 			(effects
@@
 			)
 		)
-		(property "Footprint" "Connector_PinHeader_2.54mm:PinHeader_1x03_P2.54mm_Vertical"
+		(property "Footprint" "Project_Footprints:PinHeader_1x03_P2.54mm_Vertical"
 			(at 156.21 50.8 0)
 			(effects
@@
 			)
 		)
-		(property "Footprint" "Connector_PinHeader_2.54mm:PinHeader_1x03_P2.54mm_Vertical"
+		(property "Footprint" "Project_Footprints:PinHeader_1x03_P2.54mm_Vertical"
 			(at 123.19 50.8 0)
 			(effects
@@
 			)
 		)
-		(property "Footprint" "Package_SO:MSOP-8_3x3mm_P0.65mm"
+		(property "Footprint" "Project_Footprints:MSOP-8_3x3mm_P0.65mm"
 			(at 109.22 140.97 0)
 			(effects
@@
 			)
 		)
-		(property "Footprint" "Connector_PinHeader_2.54mm:PinHeader_1x03_P2.54mm_Vertical"
+		(property "Footprint" "Project_Footprints:PinHeader_1x03_P2.54mm_Vertical"
 			(at 142.24 83.82 0)
 			(effects
@@
 			)
 		)
-		(property "Footprint" "Button_Switch_THT:SW_PUSH_6mm"
+		(property "Footprint" "Project_Footprints:SW_PUSH_6mm"
 			(at 213.36 123.19 0)
 			(effects
@@
 			)
 		)
-		(property "Footprint" "Button_Switch_THT:SW_PUSH_6mm"
+		(property "Footprint" "Project_Footprints:SW_PUSH_6mm"
 			(at 196.85 123.19 0)
 			(effects
