File: OutputMosfets.kicad_sch (KiCad schematic)
At the start: 60 parts, among them J10 Screw_Terminal_01x02, J11 Screw_Terminal_01x02, J12 Screw_Terminal_01x02, J15 Screw_Terminal_01x02, J6 Screw_Terminal_01x02, J9 Screw_Terminal_01x02, Q1 QM6006D, Q2 QM6006D, Q3 IRLZ44N, Q31 IRLZ44N, Q32 IRLZ44N, Q33 IRLZ44N, Q34 IRLZ44N, Q35 IRLZ44N, Q4 QM6006D, Q5 QM6006D, Q7 QM6006D

Commit message: Release 1.0
Other:
- note added: "LEDs at each output are driven by VDC, which can be lower than VDC2. Use VDC2>VDC if loads require higher voltage."
- note added: "Use IRLZ44N TO-220 OR the SMT N channel MOSFETs (QM6006D or whatever N Channel SMD transistor you can find that matches the pins). The board allows you to choose one type of MOSFET for each output, so you can use a TO-220 through hole, OR a DPAK TO-252 MOSFET, OR a TO-263 MOSFET (the larger variants)"
Changed lines of the file:
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@@
 	(text "OUTPUT block"
 		(exclude_from_sim no)
-		(at 163.322 24.638 0)
+		(at 121.666 21.336 0)
 		(effects
 			(font
@@
 		)
 	)
+	(text "Use IRLZ44N TO-220 OR the SMT N channel MOSFETs (QM6006D or whatever\nN Channel SMD transistor you can find that matches the pins).\nThe board allows you to choose one type of MOSFET for each output,\nso you can use a TO-220 through hole, OR a DPAK TO-252 MOSFET, OR\na TO-263 MOSFET (the larger variants)"
+		(exclude_from_sim no)
+		(at 160.02 26.162 0)
+		(effects
+			(font
+				(size 2.032 2.032)
+				(thickness 1.016)
+				(bold yes)
+			)
+			(justify left)
+		)
+	)
+	(text "LEDs at each output are driven by VDC, \nwhich can be lower than VDC2.\nUse VDC2>VDC if loads require higher voltage."
+		(exclude_from_sim no)
+		(at 192.278 173.99 0)
+		(effects
+			(font
+				(size 2.54 2.54)
+				(thickness 0.508)
+				(bold yes)
+			)
+			(justify left)
+		)
+	)

Commit message: Release 1.2
Parts:
- 2N3904_13, 2N3904_14, 2N3904_17, 2N3904_18, Q_11, Tr1: footprint TO220:TO-92_Expanded -> Project_Footprints:TO-92_Expanded
- D1, D2, D3, D4, D5, D6: footprint LED_SMD:LED_1206_3216Metric_Pad1.42x1.75mm_HandSolder -> Project_Footprints:LED_1206_3216Metric_Pad1.42x1.75mm_HandSolder
- Flyback1, Flyback2, Flyback3, Flyback4, Flyback5, Flyback6: footprint Diode_THT:D_DO-41_SOD81_P10.16mm_Horizontal -> Project_Footprints:D_DO-41_SOD81_P10.16mm_Horizontal
- J10, J11, J12, J6, J9: footprint TO220:TerminalBlock_CLEAN_2PIN -> Project_Footprints:TerminalBlock_CLEAN_2PIN
- J15: footprint TerminalBlock:TerminalBlock_bornier-2_P5.08mm -> Project_Footprints:TerminalBlock_bornier-2_P5.08mm
- Q1, Q2, Q4, Q5, Q7, Q_12: footprint termocuplu:TO-263-2_Extended -> Project_Footprints:TO-263-2_Extended
- Q3, Q31, Q32, Q33, Q34, Q35: footprint TO220:TO-220-3_EXTENDED -> Project_Footprints:TO-220-3_EXTENDED
- R1, R10, R11, R12, R13, R14, R15, R16, R17, R18, R2, R3, R4, R5, R53, R54, R55, R56, R57, R58, R6, R7, R8, R9: footprint TO220:R_Axial_Clean -> Project_Footprints:R_Axial_Clean
