File: Power.kicad_sch (KiCad schematic)
At the start: 10 parts, among them J1 DC_PowerIn, J14 Screw_Terminal_01x02, J8 Screw_Terminal_01x02, U7 LM78M05_TO252

Commit message: Release 1.0
Other:
- note added: "VDC2 is the voltage driving the loads. VDC is the input voltage powering the board. VDC2 can be higher than VDC but not higher than what the MOSFETS can withstand from drain to gate. If you use the same, then you need to solder the VDC2 to VDC pins on these screw terminals. GND is already common to both. USE only one regulator"
- note removed: "Gate driving connection options --------------------------------- 1) Gate drive soldered gate drive_HI - if the MOSFETS are logic level, no socket connectors 2) Gate drive pin to gate driver IC (requires gate driver IC) 3) Gate drive to BJT totem pole,requires PNP and NPN transistors 4) With sockets, gate drive signals go to shield and come back to gate drive_HI Output overvoltage protection opti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"
- note removed: "VDC2 is the voltage driving the loads. VDC is the input voltage powering the board. VDC2 can be higher than VDC but not higher than the Schottky diodes' breakdown voltage. If you use the same, then you need to solder the VDC2 to VDC pins on these screw terminals. GND is already common to both."
Changed lines of the file:
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@@
 	(generator_version "9.0")
 	(paper "A4")
-	(text "Gate driving connection options\n---------------------------------\n1) Gate drive soldered gate drive_HI - if the MOSFETS are logic level,\nno socket connectors\n2) Gate drive pin to gate driver IC (requires gate driver IC)\n3) Gate drive to BJT totem pole,requires PNP and NPN transistors\n4) With sockets, gate drive signals go to shield and come back to gate drive_HI\n\nOutput overvoltage protection options for inductive loads\n----------------------------------------------------------\n1) Overvoltage protection diode in series with discharge load - to VCC\n2) high voltage diode - to load or to capacitor in parallel with discharge \n   load to VCC\n\n\n"
-		(exclude_from_sim no)
-		(at 230.886 140.208 0)
-		(effects
-			(font
-				(size 1.27 1.27)
-			)
-		)
-	)
 	(text "Should be an AMS1117 3V3 for ESP32"
 		(exclude_from_sim no)
@@
 	(text "POWER Block"
 		(exclude_from_sim no)
-		(at 116.586 93.472 0)
+		(at 155.194 93.726 0)
 		(effects
 			(font
@@
 		)
 	)
-	(text "VDC2 is the voltage driving the loads.\nVDC is the input voltage powering the board.\nVDC2 can be higher than VDC but not higher than the Schottky\ndiodes' breakdown voltage.\nIf you use the same, then you need to solder\nthe VDC2 to VDC pins on these screw terminals.\nGND is already common to both."
+	(text "VDC2 is the voltage driving the loads.\nVDC is the input voltage powering the board.\nVDC2 can be higher than VDC but not higher than what the MOSFETS\ncan withstand from drain to gate.\nIf you use the same, then you need to solder\nthe VDC2 to VDC pins on these screw terminals.\nGND is already common to both.\n\n\nUSE only one regulator"
 		(exclude_from_sim no)
-		(at 81.026 79.756 0)
+		(at 84.074 85.852 0)
 		(effects
 			(font

Commit message: Release 1.2
Parts:
- AMS11173V3: footprint Package_TO_SOT_THT:TO-220-3_Horizontal_TabDown -> Project_Footprints:TO-220-3_Horizontal_TabDown
- C1, C4: footprint Capacitor_SMD:CP_Elec_6.3x3.9 -> Project_Footprints:CP_Elec_6.3x3.9
- C2, C3: footprint Capacitor_THT:C_Rect_L7.0mm_W3.5mm_P5.00mm -> Project_Footprints:C_Rect_L7.0mm_W3.5mm_P5.00mm
- J1: footprint Connector_BarrelJack:BarrelJack_Horizontal -> Project_Footprints:BarrelJack_Horizontal
- J14: footprint TerminalBlock:TerminalBlock_bornier-2_P5.08mm -> Project_Footprints:TerminalBlock_bornier-2_P5.08mm
- J8: footprint TO220:TerminalBlock_CLEAN_2PIN -> Project_Footprints:TerminalBlock_CLEAN_2PIN
- TO_220Wiring1: footprint Connector_PinSocket_2.54mm:PinSocket_1x03_P2.54mm_Vertical -> Project_Footprints:PinHeader_1x03_P2.54mm_Vertical
- U7: footprint Package_TO_SOT_SMD:TO-252-2 -> Project_Footprints:TO-252-2
Changed lines of the file:
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@@
 			)
 		)
-		(property "Footprint" "Connector_BarrelJack:BarrelJack_Horizontal"
+		(property "Footprint" "Project_Footprints:BarrelJack_Horizontal"
 			(at 31.75 26.67 0)
 			(effects
@@
 			)
 		)
-		(property "Footprint" "Package_TO_SOT_SMD:TO-252-2"
+		(property "Footprint" "Project_Footprints:TO-252-2"
 			(at 130.81 62.865 0)
 			(effects
@@
 			)
 		)
-		(property "Footprint" "TO220:TerminalBlock_CLEAN_2PIN"
+		(property "Footprint" "Project_Footprints:TerminalBlock_CLEAN_2PIN"
 			(at 40.64 60.96 0)
 			(effects
@@
 			)
 		)
-		(property "Footprint" "Capacitor_SMD:CP_Elec_6.3x3.9"
+		(property "Footprint" "Project_Footprints:CP_Elec_6.3x3.9"
 			(at 160.9852 45.72 0)
 			(effects
@@
 			)
 		)
-		(property "Footprint" "Capacitor_SMD:CP_Elec_6.3x3.9"
+		(property "Footprint" "Project_Footprints:CP_Elec_6.3x3.9"
 			(at 101.2952 48.26 0)
 			(effects
@@
 			)
 		)
-		(property "Footprint" "Connector_PinSocket_2.54mm:PinSocket_1x03_P2.54mm_Vertical"
+		(property "Footprint" "Project_Footprints:PinHeader_1x03_P2.54mm_Vertical"
 			(at 132.08 48.26 0)
 			(effects
@@
 			)
 		)
-		(property "Footprint" "Package_TO_SOT_THT:TO-220-3_Horizontal_TabDown"
+		(property "Footprint" "Project_Footprints:TO-220-3_Horizontal_TabDown"
 			(at 149.86 34.29 0)
 			(effects
@@
 			)
 		)
-		(property "Footprint" "TerminalBlock:TerminalBlock_bornier-2_P5.08mm"
+		(property "Footprint" "Project_Footprints:TerminalBlock_bornier-2_P5.08mm"
 			(at 40.64 52.07 0)
 			(effects
@@
 			)
 		)
-		(property "Footprint" "Capacitor_THT:C_Rect_L7.0mm_W3.5mm_P5.00mm"
+		(property "Footprint" "Project_Footprints:C_Rect_L7.0mm_W3.5mm_P5.00mm"
 			(at 150.8252 45.72 0)
 			(effects
@@
 			)
 		)
-		(property "Footprint" "Capacitor_THT:C_Rect_L7.0mm_W3.5mm_P5.00mm"
+		(property "Footprint" "Project_Footprints:C_Rect_L7.0mm_W3.5mm_P5.00mm"
 			(at 110.1852 48.26 0)
 			(effects
